File: pcb/hatchet36lp_pcb.kicad_pcb (KiCad board)
At the start: 2 copper layers, 179.6 x 81.6 mm, 81 parts, among them J1 Conn_01x02_Female, J2 Conn_01x02_Female, J3 Conn_01x04_Female, SW1 SW_Push, SW10 SW_Push, SW11 SW_Push, SW12 SW_Push, SW13 SW_Push, SW14 SW_Push, SW15 SW_Push, SW16 SW_Push, SW17 SW_Push, SW18 SW_Push, SW19 SW_Push, SW2 SW_Push, SW20 SW_Push, SW21 SW_Push, SW22 SW_Push, SW23 SW_Push, SW24 SW_Push, SW25 SW_Push, SW26 SW_Push, SW27 SW_Push, SW28 SW_Push, SW29 SW_Push, SW3 SW_Push, SW30 SW_Push, SW31 SW_Push, SW32 SW_Push, SW33 SW_Push, SW34 SW_Push, SW35 SW_Push, SW36 SW_Push, SW37 SW_Push, SW38 SW_SPDT, SW4 SW_Push, SW5 SW_Push, SW6 SW_Push, SW7 SW_Push, SW8 SW_Push, SW9 SW_Push, U1 BL652

Commit message: modify pin
Connections:
- U1 pad 10: unconnected-(U1-Pad10) -> /col8
- U1 pad 12: unconnected-(U1-Pad12) -> /col6
- U1 pad 13: /col6 -> unconnected-(U1-Pad13)
- U1 pad 15: /col5 -> unconnected-(U1-Pad15)
- U1 pad 17: /col4 -> /col5
- U1 pad 18: /col3 -> /col4
- U1 pad 19: unconnected-(U1-Pad19) -> /col3
- U1 pad 28: /row2 -> unconnected-(U1-Pad28)
- U1 pad 30: /col0 -> /row2
- U1 pad 32: /row1 -> /col0
- U1 pad 33: unconnected-(U1-Pad33) -> /row1
- U1 pad 7: /col9 -> unconnected-(U1-Pad7)
- U1 pad 8: unconnected-(U1-Pad8) -> /row3
- U1 pad 9: /col8 -> /col9
Routing:
- net /row3: track 93.8 -> 110.2 mm
- net /col9: track 180.2 -> 184.4 mm
- net /col3: track 90.9 -> 94.8 mm
- net /row2: track 191.3 -> 193.0 mm
- net /col4: track 107.4 -> 108.9 mm
- net /col5: track 124.4 -> 125.4 mm
- net /col0: track 54.0 -> 54.6 mm
