File: pcb/hatchet36lp_pcb.kicad_sch (KiCad schematic)
At the start: 81 parts, among them J1 Conn_01x02_Female, J2 Conn_01x02_Female, J3 Conn_01x04_Female, SW1 SW_Push, SW10 SW_Push, SW11 SW_Push, SW12 SW_Push, SW13 SW_Push, SW14 SW_Push, SW15 SW_Push, SW16 SW_Push, SW17 SW_Push, SW18 SW_Push, SW19 SW_Push, SW2 SW_Push, SW20 SW_Push, SW21 SW_Push, SW22 SW_Push, SW23 SW_Push, SW24 SW_Push, SW25 SW_Push, SW26 SW_Push, SW27 SW_Push, SW28 SW_Push, SW29 SW_Push, SW3 SW_Push, SW30 SW_Push, SW31 SW_Push, SW32 SW_Push, SW33 SW_Push, SW34 SW_Push, SW35 SW_Push, SW36 SW_Push, SW37 SW_Push, SW4 SW_Push, SW5 SW_Push, SW6 SW_Push, SW7 SW_Push, SW8 SW_Push, SW9 SW_Push, U1 BL652

Commit message: modify pin
Parts:
- J1, J2: footprint (none) -> Connector_PinHeader_2.00mm:PinHeader_1x02_P2.00mm_Vertical
- SW38: value (none) -> SW_SPDT; footprint (none) -> locallib:SW_Slide_1P2T_CK_OS102011MS2Q_SmallPad
Connections:
- net col0: now also U1.32 (SIO_31/AIN7); no longer U1.30 (SIO_17)
- net col3: now also U1.19 (SIO_06); no longer U1.18 (SIO_07)
- net col4: now also U1.18 (SIO_07); no longer U1.17 (SIO_08)
- net col5: now also U1.17 (SIO_08); no longer U1.15 (SIO_09/NFC1)
- net col6: now also U1.12 (SIO_12); no longer U1.13 (SIO_11)
- net col8: now also U1.10 (SIO_16); no longer U1.9 (SIO_18)
- net col9: now also U1.9 (SIO_18); no longer U1.7 (SIO_21)
- net row1: now also U1.33 (SIO_30/AIN6); no longer U1.32 (SIO_31/AIN7)
- net row2: now also U1.30 (SIO_17); no longer U1.28 (SIO_13)
- net row3: now also U1.8 (SIO_20)
- no-connect marks 19 -> 18
Changed lines of the file:
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@@
   (junction (at 166.37 46.99) (diameter 0) (color 0 0 0 0)
   )
-  (no_connect (at 211.455 142.24))
   (no_connect (at 262.255 142.24))
-  (no_connect (at 262.255 139.7))
   (no_connect (at 262.255 134.62))
   (no_connect (at 262.255 132.08))
@@
   (no_connect (at 262.255 121.92))
   (no_connect (at 262.255 119.38))
-  (no_connect (at 262.255 114.3))
   (no_connect (at 211.455 111.76))
-  (no_connect (at 211.455 116.84))
   (no_connect (at 211.455 127))
-  (no_connect (at 211.455 132.08))
-  (no_connect (at 211.455 139.7))
   (no_connect (at 211.455 106.68))
   (no_connect (at 211.455 101.6))
+  (no_connect (at 211.455 124.46))
   (no_connect (at 99.695 123.825))
+  (no_connect (at 262.255 137.16))
+  (no_connect (at 211.455 139.7))
+  (no_connect (at 211.455 134.62))
+  (no_connect (at 211.455 129.54))
   (wire (pts (xy 92.075 130.81) (xy 80.01 130.81))
     (stroke (width 0) (type default) (color 0 0 0 0))
@@
   (label "col0" (at 33.02 16.51 90)
     (effects (font (size 1.27 1.27)) (justify left bottom))
+  )
+  (label "col5" (at 211.455 121.92 180)
+    (effects (font (size 1.27 1.27)) (justify right bottom))
+  )
+  (label "col6" (at 211.455 132.08 180)
+    (effects (font (size 1.27 1.27)) (justify right bottom))
   )
   (label "col1" (at 211.455 109.22 180)
@@
     (effects (font (size 1.27 1.27)) (justify right bottom))
   )
-  (label "col9" (at 262.255 137.16 0)
-    (effects (font (size 1.27 1.27)) (justify left bottom))
-  )
   (label "col2" (at 71.12 16.51 90)
     (effects (font (size 1.27 1.27)) (justify left bottom))
   )
-  (label "col0" (at 211.455 144.78 180)
-    (effects (font (size 1.27 1.27)) (justify right bottom))
+  (label "col0" (at 262.255 111.76 0)
+    (effects (font (size 1.27 1.27)) (justify left bottom))
   )
   (label "col6" (at 147.32 16.51 90)
@@
     (effects (font (size 1.27 1.27)) (justify right bottom))
   )
-  (label "row2" (at 211.455 134.62 180)
+  (label "SWDCLK" (at 262.255 101.6 0)
+    (effects (font (size 1.27 1.27)) (justify left bottom))
+  )
+  (label "col4" (at 109.22 16.51 90)
+    (effects (font (size 1.27 1.27)) (justify left bottom))
+  )
+  (label "row2" (at 211.455 144.78 180)
     (effects (font (size 1.27 1.27)) (justify right bottom))
   )
-  (label "SWDCLK" (at 262.255 101.6 0)
-    (effects (font (size 1.27 1.27)) (justify left bottom))
-  )
-  (label "col4" (at 109.22 16.51 90)
-    (effects (font (size 1.27 1.27)) (justify left bottom))
-  )
   (label "col8" (at 185.42 16.51 90)
     (effects (font (size 1.27 1.27)) (justify left bottom))
   )
-  (label "col8" (at 262.255 144.78 0)
-    (effects (font (size 1.27 1.27)) (justify left bottom))
-  )
-  (label "row1" (at 262.255 111.76 0)
+  (label "col4" (at 211.455 119.38 180)
+    (effects (font (size 1.27 1.27)) (justify right bottom))
+  )
+  (label "col9" (at 262.255 144.78 0)
+    (effects (font (size 1.27 1.27)) (justify left bottom))
+  )
+  (label "col3" (at 211.455 116.84 180)
+    (effects (font (size 1.27 1.27)) (justify right bottom))
+  )
+  (label "row1" (at 262.255 114.3 0)
     (effects (font (size 1.27 1.27)) (justify left bottom))
   )
@@
     (effects (font (size 1.27 1.27)) (justify right bottom))
   )
+  (label "col8" (at 211.455 142.24 180)
+    (effects (font (size 1.27 1.27)) (justify right bottom))
+  )
   (label "SWDIO" (at 138.43 161.925 180)
     (effects (font (size 1.27 1.27)) (justify right bottom))
@@
     (effects (font (size 1.27 1.27)) (justify left bottom))
   )
-  (label "col6" (at 211.455 129.54 180)
-    (effects (font (size 1.27 1.27)) (justify right bottom))
-  )
   (label "col7" (at 211.455 137.16 180)
     (effects (font (size 1.27 1.27)) (justify right bottom))
@@
     (effects (font (size 1.27 1.27)) (justify left bottom))
   )
+  (label "row3" (at 262.255 139.7 0)
+    (effects (font (size 1.27 1.27)) (justify left bottom))
+  )
   (label "col5" (at 128.27 16.51 90)
     (effects (font (size 1.27 1.27)) (justify left bottom))
-  )
-  (label "col3" (at 211.455 119.38 180)
-    (effects (font (size 1.27 1.27)) (justify right bottom))
   )
   (label "row3" (at 20.32 92.71 180)
@@
   (label "SWDIO" (at 262.255 104.14 0)
     (effects (font (size 1.27 1.27)) (justify left bottom))
-  )
-  (label "col5" (at 211.455 124.46 180)
-    (effects (font (size 1.27 1.27)) (justify right bottom))
-  )
-  (label "col4" (at 211.455 121.92 180)
-    (effects (font (size 1.27 1.27)) (justify right bottom))
   )
   (label "col2" (at 211.455 114.3 180)
@@
       (effects (font (size 1.27 1.27)) (justify left))
     )
-    (property "Footprint" "" (id 2) (at 97.155 147.955 0)
+    (property "Footprint" "Connector_PinHeader_2.00mm:PinHeader_1x02_P2.00mm_Vertical" (id 2) (at 97.155 147.955 0)
       (effects (font (size 1.27 1.27)) hide)
     )
@@
       (effects (font (size 1.27 1.27)) (justify left))
     )
-    (property "Footprint" "" (id 2) (at 97.155 156.21 0)
+    (property "Footprint" "Connector_PinHeader_2.00mm:PinHeader_1x02_P2.00mm_Vertical" (id 2) (at 97.155 156.21 0)
       (effects (font (size 1.27 1.27)) hide)
     )
@@
     (in_bom yes) (on_board yes) (fields_autoplaced)
     (property "Reference" "SW38" (id 0) (at 94.615 113.03 0))
-    (property "Value" "" (id 1) (at 94.615 115.57 0))
-    (property "Footprint" "" (id 2) (at 94.615 121.285 0)
-      (effects (font (size 1.27 1.27)) hide)
-    )
+    (property "Value" "SW_SPDT" (id 1) (at 94.615 115.57 0))
+    (property "Footprint" "locallib:SW_Slide_1P2T_CK_OS102011MS2Q_SmallPad" (id 2) (at 94.615 121.285 0)
+      (effects (font (size 1.27 1.27)) hide)
+    )
